File: jeff-orTHo.kicad_pcb (KiCad board)
At the start: 2 copper layers, 106 parts, among them SW1 SW_Push, U1 ATmega32U4-AU, Y1 Crystal_GND24_Small

Commit message: Routing
Layout tweaks, need ground/power fills
Parts:
- added H1: MountingHole, MountingHole:MountingHole_2.2mm_M2, B.Cu at (-92.1, 42.9)
- added H2: MountingHole, MountingHole:MountingHole_2.2mm_M2, B.Cu at (-82.5, 81.0)
- added H3: MountingHole, MountingHole:MountingHole_2.2mm_M2, B.Cu at (-34.9, 42.9)
- added H4: MountingHole, MountingHole:MountingHole_2.2mm_M2, B.Cu at (-25.4, 81.0)
- added H5: MountingHole, MountingHole:MountingHole_2.2mm_M2, B.Cu at (41.3, 42.9)
- added H6: MountingHole, MountingHole:MountingHole_2.2mm_M2, B.Cu at (31.8, 81.0)
- added H7: MountingHole, MountingHole:MountingHole_2.2mm_M2, B.Cu at (98.4, 42.9)
- added H8: MountingHole, MountingHole:MountingHole_2.2mm_M2, B.Cu at (88.9, 81.0)
- MX101, MX102, MX103, MX104, MX105, MX106, MX107, MX108, MX109, MX110, MX111, MX112, MX201, MX202, MX203, MX204, MX205, MX206, MX207, MX208, MX209, MX210, MX211, MX212, MX301, MX302, MX303, MX304, MX305, MX306, MX307, MX308, MX309, MX310, MX311, MX312: footprint MX_Alps_Hybrid:MX-1U -> MX_Alps_Hybrid:MX-1U-NoLED
- MX401, MX403, MX404, MX406, MX407, MX409, MX410, MX412: footprint MX_Alps_Hybrid:MX-1.5U -> MX_Alps_Hybrid:MX-1.5U-NoLED
- moved SW1 128.0 mm to (-119.9, 69.0)
- moved R1 126.0 mm to (-126.6, 63.1), turned to 270 degrees
- moved R2 122.7 mm to (-121.5, 33.7)
- moved R3 122.7 mm to (-119.0, 33.7)
- moved R6 122.7 mm to (-124.1, 33.7)
- moved USB1 122.6 mm to (-120.3, 30.0)
- moved C2 121.5 mm to (-124.0, 63.1), turned to 270 degrees
- moved C3 120.9 mm to (-127.5, 54.0), turned to 90 degrees
- moved R5 120.2 mm to (-113.9, 33.7)
- moved C7 117.5 mm to (-127.5, 47.1), turned to 270 degrees
- moved Y1 114.3 mm to (-119.9, 63.1), turned to 180 degrees
- moved F1 112.7 mm to (-116.5, 33.7)
- moved C4 112.6 mm to (-116.5, 42.9)
- moved C1 107.2 mm to (-115.7, 63.1), turned to 90 degrees
- moved U1 104.1 mm to (-119.5, 52.3), turned to 0 degrees
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Connections:
- U1 pad 21: Net-(U1-Pad21) -> ROW3
- U1 pad 22: Net-(U1-Pad22) -> ROW2
- U1 pad 25: Net-(U1-Pad25) -> COL5
- U1 pad 26: Net-(U1-Pad26) -> COL6
- U1 pad 27: Net-(U1-Pad27) -> COL7
- U1 pad 28: Net-(U1-Pad28) -> COL8
- U1 pad 29: Net-(U1-Pad29) -> COL9
- U1 pad 30: Net-(U1-Pad30) -> COL10
- U1 pad 31: Net-(U1-Pad31) -> COL11
- U1 pad 32: Net-(U1-Pad32) -> ROW1
- U1 pad 36: Net-(U1-Pad36) -> COL4
- U1 pad 37: Net-(U1-Pad37) -> COL3
- U1 pad 38: Net-(U1-Pad38) -> COL2
- U1 pad 39: Net-(U1-Pad39) -> COL1
- U1 pad 40: Net-(U1-Pad40) -> ROW0
- U1 pad 41: Net-(U1-Pad41) -> COL0
Routing:
- net COL11: track 0.00 -> 275.9 mm, vias 0 -> 2
- net ROW3: track 0.00 -> 259.8 mm, vias 0 -> 1
- net ROW2: track 0.00 -> 250.2 mm, vias 0 -> 1
- net ROW0: track 0.00 -> 249.8 mm, vias 0 -> 1
- net ROW1: track 0.00 -> 238.8 mm, vias 0 -> 1
- net COL9: track 0.00 -> 238.5 mm, vias 0 -> 2
- net COL10: track 0.00 -> 237.6 mm, vias 0 -> 2
- net COL8: track 0.00 -> 218.0 mm, vias 0 -> 2
- net COL6: track 0.00 -> 180.7 mm, vias 0 -> 2
- net COL7: track 0.00 -> 179.8 mm, vias 0 -> 2
- net COL5: track 0.00 -> 160.4 mm, vias 0 -> 2
- net COL3: track 0.00 -> 132.1 mm, vias 0 -> 2
- net COL4: track 0.00 -> 129.7 mm, vias 0 -> 2
- net COL2: track 0.00 -> 112.9 mm, vias 0 -> 2
- net COL0: track 0.00 -> 78.8 mm, vias 0 -> 2
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Other:
- net class Default: clearance 0.2 -> 0.2032; trace_width 0.25 -> 0.254; via_dia 0.8 -> 0.8128; via_drill 0.4 -> 0.4064
- net class Power added: clearance 0.2032, trace_width 0.381, via_dia 0.8128, via_drill 0.4064
- rule trace_clearance: 0.2 -> 0.2032
