File: jeff-orTHo.sch (KiCad schematic (older format))
At the start: 106 parts, among them SW1 SW_Push, U1 ATmega32U4-AU, Y1 Crystal_GND24_Small

Commit message: Initial layout
Parts:
- C7: footprint Diode_SMD:D_SOD-123 -> Capacitor_SMD:C_1206_3216Metric_Pad1.33x1.80mm_HandSolder
- F1: footprint MX_Alps_Hybrid:MX-1U -> Fuse:Fuse_1206_3216Metric_Pad1.42x1.75mm_HandSolder
Changed lines of the file:
@@
 F 0 "C7" H 1909 4104 50  0000 R CNN
 F 1 ".1u" H 1909 4195 50  0000 R CNN
-F 2 "Diode_SMD:D_SOD-123" H 2000 4150 50  0001 C CNN
+F 2 "Capacitor_SMD:C_1206_3216Metric_Pad1.33x1.80mm_HandSolder" H 2000 4150 50  0001 C CNN
 F 3 "~" H 2000 4150 50  0001 C CNN
 	1    2000 4150
@@
 F 0 "F1" V 2145 5250 50  0000 C CNN
 F 1 "500m" V 2236 5250 50  0000 C CNN
-F 2 "MX_Alps_Hybrid:MX-1U" H 2400 5050 50  0001 L CNN
+F 2 "Fuse:Fuse_1206_3216Metric_Pad1.42x1.75mm_HandSolder" H 2400 5050 50  0001 L CNN
 F 3 "~" H 2350 5250 50  0001 C CNN
 	1    2350 5250

Commit message: Routing
Layout tweaks, need ground/power fills
Parts:
- added H1, H2, H3, H4, H5, H6, H7, H8: MountingHole, MountingHole:MountingHole_2.2mm_M2, symbol Mechanical:MountingHole
- MX101, MX102, MX103, MX104, MX105, MX106, MX107, MX108, MX109, MX110, MX111, MX112, MX201, MX202, MX203, MX204, MX205, MX206, MX207, MX208, MX209, MX210, MX211, MX212, MX301, MX302, MX303, MX304, MX305, MX306, MX307, MX308, MX309, MX310, MX311, MX312: footprint MX_Alps_Hybrid:MX-1U -> MX_Alps_Hybrid:MX-1U-NoLED
- MX401, MX403, MX404, MX406, MX407, MX409, MX410, MX412: footprint MX_Alps_Hybrid:MX-1.5U -> MX_Alps_Hybrid:MX-1.5U-NoLED
Connections:
- net COL0: now also U1.41 (PF0)
- net COL1: now also U1.39 (PF4)
- net COL10: now also U1.30 (PB6)
- net COL11: now also U1.31 (PC6)
- net COL2: now also U1.38 (PF5)
- net COL3: now also U1.37 (PF6)
- net COL4: now also U1.36 (PF7)
- net COL5: now also U1.25 (PD4)
- net COL6: now also U1.26 (PD6)
- net COL7: now also U1.27 (PD7)
- net COL8: now also U1.28 (PB4)
- net COL9: now also U1.29 (PB5)
- net ROW0: now also U1.40 (PF1)
- net ROW1: now also U1.32 (PC7)
- net ROW2: now also U1.22 (PD5)
- net ROW3: now also U1.21 (PD3)
